File: ethernet.kicad_sch (KiCad schematic)
At the start: 50 parts, among them J301 JK0654219, U301 MIC33050-4YHL, U302 KSZ9031RNXCA, U303 ASDMB-25.000MHz, U304 74LVC2G07, U305 TXS0102DCU

Commit message: Place motor drivers, start layout of Ethernet PHY
Parts:
- removed C327: 0.1U, Capacitor_SMD:C_0603_1608Metric, symbol Device:C_Small
- added C312: 0.1U, Capacitor_SMD:C_0402_1005Metric, symbol Device:C_Small
- C301, C315: footprint Capacitor_SMD:C_0603_1608Metric -> Capacitor_SMD:C_0402_1005Metric
- C302: renamed from C329; footprint Capacitor_SMD:C_0603_1608Metric -> Capacitor_SMD:C_0402_1005Metric
- C303: renamed from C302; footprint Capacitor_SMD:C_0603_1608Metric -> Capacitor_SMD:C_0402_1005Metric
- C304: renamed from C330; footprint Capacitor_SMD:C_0603_1608Metric -> Capacitor_SMD:C_0402_1005Metric
- C310: renamed from C306; footprint Capacitor_SMD:C_0603_1608Metric -> Capacitor_SMD:C_0402_1005Metric
- C311: renamed from C309; footprint Capacitor_SMD:C_0603_1608Metric -> Capacitor_SMD:C_0402_1005Metric
- C313: renamed from C310; footprint Capacitor_SMD:C_0603_1608Metric -> Capacitor_SMD:C_0402_1005Metric
- C314: renamed from C311; footprint Capacitor_SMD:C_0603_1608Metric -> Capacitor_SMD:C_0402_1005Metric
- C316: renamed from C312; footprint Capacitor_SMD:C_0603_1608Metric -> Capacitor_SMD:C_0402_1005Metric
- C317: renamed from C316; footprint Capacitor_SMD:C_0603_1608Metric -> Capacitor_SMD:C_0402_1005Metric
- C318: renamed from C313; footprint Capacitor_SMD:C_0603_1608Metric -> Capacitor_SMD:C_0402_1005Metric
- C319: renamed from C314; footprint Capacitor_SMD:C_0603_1608Metric -> Capacitor_SMD:C_0402_1005Metric
- C320: renamed from C317; footprint Capacitor_SMD:C_0603_1608Metric -> Capacitor_SMD:C_0402_1005Metric
- C321: renamed from C318; footprint Capacitor_SMD:C_0603_1608Metric -> Capacitor_SMD:C_0402_1005Metric
- C322: renamed from C319; footprint Capacitor_SMD:C_0603_1608Metric -> Capacitor_SMD:C_0402_1005Metric
- C323: renamed from C321; footprint Capacitor_SMD:C_0603_1608Metric -> Capacitor_SMD:C_0402_1005Metric
- C324: renamed from C320; footprint Capacitor_SMD:C_0603_1608Metric -> Capacitor_SMD:C_0402_1005Metric
- C325: renamed from C322; footprint Capacitor_SMD:C_0603_1608Metric -> Capacitor_SMD:C_0402_1005Metric
- C327: renamed from C323; footprint Capacitor_SMD:C_0603_1608Metric -> Capacitor_SMD:C_0402_1005Metric
- C328: renamed from C324; footprint Capacitor_SMD:C_0603_1608Metric -> Capacitor_SMD:C_0402_1005Metric
- C329: renamed from C326; footprint Capacitor_SMD:C_0603_1608Metric -> Capacitor_SMD:C_0402_1005Metric
- C330: renamed from C328; footprint Capacitor_SMD:C_0603_1608Metric -> Capacitor_SMD:C_0402_1005Metric
- renumbered C303 to C305, C304 to C306, C305 to C307, C307 to C308, C308 to C309, C325 to C326, U305 to U302, U302 to U303, U303 to U304, U304 to U305
Connections:
- net +1V8: now also C312.1
- net ETHERNET.MDC: now also U302.4 (A2); no longer U302.5 (A1)
- net ETHERNET.MDIO: now also U302.5 (A1); no longer U302.4 (A2)
- net GND: now also C312.2
- net MDC: now also U302.1 (B2); no longer U302.8 (B1)
- net MDIO: now also U302.8 (B1); no longer U302.1 (B2)
- net CFF: now reaches C303.2, U301.11 (CFF)
- no-connect marks 2 -> 3
Other:
- moved on the sheet: C303, C305, C306, C307, C308, C309, C310, C311, FB301, FB302

Commit message: Add FTDI chip
Parts:
- renumbered C301 to C401, C302 to C402, C303 to C403, C304 to C404, C305 to C405, C306 to C406, C307 to C407, C308 to C408, C309 to C409, C310 to C410, C311 to C411, C312 to C412, C313 to C413, C314 to C414, C315 to C415, C316 to C416, C317 to C417, C318 to C418, C319 to C419, C320 to C420, C321 to C421, C322 to C422, C323 to C423, C324 to C424, C325 to C425, C326 to C426, C327 to C427, C328 to C428, C329 to C429, C330 to C430, D301 to D401, D302 to D402, FB301 to FB401, FB302 to FB402, FB303 to FB403, J301 to J401, R301 to R401, R302 to R402, R303 to R403, R304 to R404, R305 to R405, R306 to R406, R307 to R407, R308 to R408, R309 to R409, U301 to U401, U302 to U402, U303 to U403, U304 to U404, U305 to U405

Commit message: Connect Ethernet PHY to FPGA, route RGMII signals
Parts:
- removed C402, C404: 0.1u, Capacitor_SMD:C_0402_1005Metric, symbol Device:C_Small
- removed U402: TXS0102DCU, Package_SO:VSSOP-8_2.3x2mm_P0.5mm, symbol Logic_LevelTranslator:TXS0102DCU
- C401: footprint Capacitor_SMD:C_0402_1005Metric -> Capacitor_SMD:C_0603_1608Metric
- C402: renamed from C403; footprint Capacitor_SMD:C_0402_1005Metric -> Capacitor_SMD:C_0603_1608Metric
- C408: renamed from C410; value 0.1U -> 0.1u
- C409: renamed from C411; value 0.1U -> 0.1u
- C410: renamed from C412; value 0.1U -> 0.1u
- C411: renamed from C413; value 0.1U -> 0.1u
- C412: renamed from C414; value 0.1U -> 0.1u
- C413: renamed from C415; value 0.1U -> 0.1u
- C414: renamed from C416; value 0.1U -> 0.1u
- C415: renamed from C417; value 0.1U -> 0.1u
- C416: renamed from C418; value 0.1U -> 0.1u
- C417: renamed from C419; value 0.1U -> 0.1u
- C418: renamed from C420; value 0.1U -> 0.1u
- C419: renamed from C421; value 0.1U -> 0.1u
- C420: renamed from C422; value 0.1U -> 0.1u
- C421: renamed from C423; value 0.1U -> 0.1u
- C422: renamed from C424; footprint Capacitor_SMD:C_0402_1005Metric -> Capacitor_SMD:C_0603_1608Metric
- C423: renamed from C425; footprint Capacitor_SMD:C_0402_1005Metric -> Capacitor_SMD:C_0603_1608Metric
- C425: renamed from C427; footprint Capacitor_SMD:C_0402_1005Metric -> Capacitor_SMD:C_0603_1608Metric
- C426: renamed from C428; footprint Capacitor_SMD:C_0402_1005Metric -> Capacitor_SMD:C_0603_1608Metric
- C427: renamed from C429; footprint Capacitor_SMD:C_0402_1005Metric -> Capacitor_SMD:C_0603_1608Metric
- C428: renamed from C430; footprint Capacitor_SMD:C_0402_1005Metric -> Capacitor_SMD:C_0603_1608Metric
- R403, R405: footprint Resistor_SMD:R_0603_1608Metric -> Resistor_SMD:R_0402_1005Metric
- renumbered C405 to C403, C406 to C404, C407 to C405, C408 to C406, C409 to C407, C426 to C424, U403 to U402, U404 to U403, U405 to U404
Connections:
- net +1V8 is gone; now on net +3V3: C405.1, C408.1, C409.1, C410.1, D401.1 (K), R401.1, R402.1, R404.1, R407.1, U402.16 (DVDDH), U402.34 (DVDDH), U402.40 (DVDDH), U404.5 (VCC), U404.5 (VCC)
- net MDC is gone; now on net ETHERNET.MDC: U402.36 (MDC)
- net MDIO is gone; now on net ETHERNET.MDIO: R404.2, U402.37 (MDIO)
- net LED1: now also U404.3; no longer U404.1
- net LED1K: now also U404.4; no longer U404.6
- net LED2: now also U404.1; no longer R402.2, U402.38 (INT_N/PME_N2), U404.3
- net LED2K: now also U404.6; no longer U404.4
- net CT1: now reaches C428.1, J401.12 (MXCT1)
- net CT3: now reaches C426.1, J401.1 (MXCT3)
- net LED_MODE: now reaches R401.2, U402.41 (CLK125_NDO/LED_MODE)
- net ISET: now reaches R406.1, U402.48 (ISET)
- net LED2A: now reaches J401.14 (LED2+), R408.1
- net CT2: now reaches C427.1, J401.6 (MXCT2)
- net CT4: now reaches C425.1, J401.7 (MXCT4)
- net LED1A: now reaches J401.16 (LED1+), R409.1
- new net ~INT~/~PME2: R402.2, U402.38 (INT_N/PME_N2)
Other:
- note removed: "MDIO and MDC signals need to be level shifted from Zynq EMIO level (3.3V) to Ethernet PHY DVDDH level (1.8V)"
- note removed: "Zynq MIO is 1.8V LVCMOS"
- moved on the sheet: C413, C415, C418, C420, C421, R406, R409, U404A, U404B
