File: ethernet.kicad_sch (KiCad schematic)
At the start: 47 parts, among them J401 JK0654219, U401 MIC33050-4YHL, U402 KSZ9031RNXCA, U403 ASDMB-25.000MHz, U404 74LVC2G07

Commit message: Attach ethernet to PL, layout and route
Parts:
- removed D401, D402: 1N4148WS, Diode_SMD:D_SOD-323, symbol Diode:1N4148WS
- added C429: 0.1u, Capacitor_SMD:C_0603_1608Metric, symbol Device:C_Small
- added D401, D402: 1N4148WT, Diode_SMD:D_SOD-523, symbol Diode:1N4148WT
- C402: footprint Capacitor_SMD:C_0603_1608Metric -> Capacitor_SMD:C_0402_1005Metric
- FB401, FB402, FB403: footprint Inductor_SMD:L_0603_1608Metric -> Inductor_SMD:L_0402_1005Metric
- R401, R402, R404, R406: footprint Resistor_SMD:R_0603_1608Metric -> Resistor_SMD:R_0402_1005Metric
Connections:
- net +3V3: now also C429.1, D401.1 (K)
- net GND: now also C422.2, U403.2 (GND), C429.2
- net LED1: now also U404.1; no longer U404.3
- net LED1K: now also U404.6; no longer U404.4
- net LED2: now also U404.3; no longer U404.1
- net LED2K: now also U404.4; no longer U404.6
- net TXRXB+: now also J401.5 (MX2-); no longer J401.4 (MX2+)
- net TXRXB-: now also J401.4 (MX2+); no longer J401.5 (MX2-)
- net TXRXD+: now also J401.9 (MX4-); no longer J401.8 (MX4+)
- net TXRXD-: now also J401.8 (MX4+); no longer J401.9 (MX4-)
- net ~RESET: now also D402.1 (K)
- net ~RESET_IN renamed ~ENET_RST
- net ~ENET_RST: now also D401.2 (A), D402.2 (A)
Other:
- note added: "Maybe put ferrites on RGMII lines?"
- note added: "The differential pairs for TXRXB and TXRXD have their polarity inverted because it makes the routing easier. The KSZ9031RNX automatically corrects for this. See KSZ9031RNX datasheet Section 3.4 "Pair-Swap, Alignment, and Polarity Check""
- moved on the sheet: C422, C423, R407, U403, U404A, U404B

Commit message: Move Ethernet around to save space
Connections:
- net TXRXB+: now also J401.4 (MX2+); no longer J401.5 (MX2-)
- net TXRXB-: now also J401.5 (MX2-); no longer J401.4 (MX2+)
- net TXRXD+: now also J401.8 (MX4+); no longer J401.9 (MX4-)
- net TXRXD-: now also J401.9 (MX4-); no longer J401.8 (MX4+)
Changed lines of the file:
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@@
-(kicad_sch (version 20200714) (host eeschema "5.99.0-unknown-a146cd9~102~ubuntu20.04.1")
+(kicad_sch (version 20200714) (host eeschema "5.99.0-unknown-9b6ade6b1~102~ubuntu20.04.1")
   (page 4 15)
   (paper "B")
@@
   (junction (at 327.66 147.32) (diameter 1.016) (color 0 0 0 0))
   (junction (at 330.2 147.32) (diameter 1.016) (color 0 0 0 0))
-  (no_connect (at 208.28 134.62))
   (no_connect (at 45.72 39.37))
   (no_connect (at 208.28 185.42))
+  (no_connect (at 208.28 134.62))
   (bus_entry (at 114.3 129.54) (size 2.54 2.54)
     (stroke (width 0.1524) (type solid) (color 0 0 0 0))
@@
     (stroke (width 0) (type solid) (color 0 0 0 0))
   )
-  (bus (pts (xy 114.3 129.54) (xy 114.3 137.16))
-    (stroke (width 0) (type solid) (color 0 0 0 0))
-  )
-  (bus (pts (xy 114.3 137.16) (xy 114.3 142.24))
-    (stroke (width 0) (type solid) (color 0 0 0 0))
-  )
-  (bus (pts (xy 114.3 142.24) (xy 114.3 144.78))
-    (stroke (width 0) (type solid) (color 0 0 0 0))
-  )
-  (bus (pts (xy 114.3 144.78) (xy 114.3 152.4))
-    (stroke (width 0) (type solid) (color 0 0 0 0))
-  )
-  (bus (pts (xy 114.3 152.4) (xy 114.3 154.94))
-    (stroke (width 0) (type solid) (color 0 0 0 0))
-  )
-  (bus (pts (xy 114.3 154.94) (xy 114.3 160.02))
-    (stroke (width 0) (type solid) (color 0 0 0 0))
-  )
-  (bus (pts (xy 114.3 160.02) (xy 114.3 165.1))
+  (bus (pts (xy 114.3 129.54) (xy 114.3 134.62))
+    (stroke (width 0) (type solid) (color 0 0 0 0))
+  )
+  (bus (pts (xy 114.3 134.62) (xy 114.3 139.7))
+    (stroke (width 0) (type solid) (color 0 0 0 0))
+  )
+  (bus (pts (xy 114.3 139.7) (xy 114.3 142.24))
+    (stroke (width 0) (type solid) (color 0 0 0 0))
+  )
+  (bus (pts (xy 114.3 142.24) (xy 114.3 147.32))
+    (stroke (width 0) (type solid) (color 0 0 0 0))
+  )
+  (bus (pts (xy 114.3 147.32) (xy 114.3 152.4))
+    (stroke (width 0) (type solid) (color 0 0 0 0))
+  )
+  (bus (pts (xy 114.3 152.4) (xy 114.3 157.48))
+    (stroke (width 0) (type solid) (color 0 0 0 0))
+  )
+  (bus (pts (xy 114.3 157.48) (xy 114.3 162.56))
+    (stroke (width 0) (type solid) (color 0 0 0 0))
+  )
+  (bus (pts (xy 114.3 162.56) (xy 114.3 165.1))
     (stroke (width 0) (type solid) (color 0 0 0 0))
   )
@@
     (effects (font (size 1.27 1.27)) (justify left bottom))
   )
-  (label "TXRXD+" (at 353.06 91.44 0)
+  (label "TXRXD-" (at 353.06 91.44 0)
     (effects (font (size 1.27 1.27)) (justify left bottom))
   )
@@
     (effects (font (size 1.27 1.27)) (justify left bottom))
   )
-  (label "TXRXD-" (at 353.06 96.52 0)
+  (label "TXRXD+" (at 353.06 96.52 0)
     (effects (font (size 1.27 1.27)) (justify left bottom))
   )
@@
     (effects (font (size 1.27 1.27)) (justify left bottom))
   )
-  (label "TXRXB+" (at 353.06 111.76 0)
+  (label "TXRXB-" (at 353.06 111.76 0)
     (effects (font (size 1.27 1.27)) (justify left bottom))
   )
@@
     (effects (font (size 1.27 1.27)) (justify left bottom))
   )
-  (label "TXRXB-" (at 353.06 116.84 0)
-    (effects (font (size 1.27 1.27)) (justify left bottom))
-  )
+  (label "TXRXB+" (at 353.06 116.84 0)
+    (effects (font (size 1.27 1.27)) (justify left bottom))
+  )

Commit message: Expand PCB, change to inches, center Snickerdoodle
Changed lines of the file:
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@@
-(kicad_sch (version 20200714) (host eeschema "5.99.0-unknown-9b6ade6b1~102~ubuntu20.04.1")
+(kicad_sch (version 20200714) (host eeschema "5.99.0-unknown-829316fad~102~ubuntu20.04.1")
   (page 4 15)
   (paper "B")
@@
   (junction (at 327.66 147.32) (diameter 1.016) (color 0 0 0 0))
   (junction (at 330.2 147.32) (diameter 1.016) (color 0 0 0 0))
+  (no_connect (at 208.28 134.62))
+  (no_connect (at 208.28 185.42))
   (no_connect (at 45.72 39.37))
-  (no_connect (at 208.28 185.42))
-  (no_connect (at 208.28 134.62))
   (bus_entry (at 114.3 129.54) (size 2.54 2.54)
     (stroke (width 0.1524) (type solid) (color 0 0 0 0))
@@
     (stroke (width 0) (type solid) (color 0 0 0 0))
   )
-  (bus (pts (xy 114.3 129.54) (xy 114.3 134.62))
-    (stroke (width 0) (type solid) (color 0 0 0 0))
-  )
-  (bus (pts (xy 114.3 134.62) (xy 114.3 139.7))
-    (stroke (width 0) (type solid) (color 0 0 0 0))
-  )
-  (bus (pts (xy 114.3 139.7) (xy 114.3 142.24))
+  (bus (pts (xy 114.3 129.54) (xy 114.3 137.16))
+    (stroke (width 0) (type solid) (color 0 0 0 0))
+  )
+  (bus (pts (xy 114.3 137.16) (xy 114.3 142.24))
     (stroke (width 0) (type solid) (color 0 0 0 0))
   )
@@
     (stroke (width 0) (type solid) (color 0 0 0 0))
   )
-  (bus (pts (xy 114.3 147.32) (xy 114.3 152.4))
-    (stroke (width 0) (type solid) (color 0 0 0 0))
-  )
-  (bus (pts (xy 114.3 152.4) (xy 114.3 157.48))
-    (stroke (width 0) (type solid) (color 0 0 0 0))
-  )
-  (bus (pts (xy 114.3 157.48) (xy 114.3 162.56))
-    (stroke (width 0) (type solid) (color 0 0 0 0))
-  )
-  (bus (pts (xy 114.3 162.56) (xy 114.3 165.1))
-    (stroke (width 0) (type solid) (color 0 0 0 0))
-  )
+  (bus (pts (xy 114.3 147.32) (xy 114.3 154.94))
+    (stroke (width 0) (type solid) (color 0 0 0 0))
+  )
+  (bus (pts (xy 114.3 154.94) (xy 114.3 160.02))
+    (stroke (width 0) (type solid) (color 0 0 0 0))
+  )
+  (bus (pts (xy 114.3 160.02) (xy 114.3 165.1))
+    (stroke (width 0) (type solid) (color 0 0 0 0))
+  )

Commit message: Move Ethernet PHY to left side of board
Parts:
- C402: Rated Voltage (none) -> 50V
- C423: footprint Capacitor_SMD:C_0603_1608Metric -> Capacitor_SMD:C_0402_1005Metric
- R407: footprint Resistor_SMD:R_0603_1608Metric -> Resistor_SMD:R_0402_1005Metric
Changed lines of the file:
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@@
-(kicad_sch (version 20200714) (host eeschema "5.99.0-unknown-829316fad~102~ubuntu20.04.1")
+(kicad_sch (version 20200828) (generator eeschema)
   (page 4 15)
   (paper "B")
@@
   (junction (at 330.2 147.32) (diameter 1.016) (color 0 0 0 0))
   (no_connect (at 208.28 134.62))
+  (no_connect (at 45.72 39.37))
   (no_connect (at 208.28 185.42))
-  (no_connect (at 45.72 39.37))
   (bus_entry (at 114.3 129.54) (size 2.54 2.54)
     (stroke (width 0.1524) (type solid) (color 0 0 0 0))
@@
     (stroke (width 0) (type solid) (color 0 0 0 0))
   )
-  (bus (pts (xy 114.3 121.92) (xy 114.3 129.54))
-    (stroke (width 0) (type solid) (color 0 0 0 0))
-  )
-  (bus (pts (xy 114.3 129.54) (xy 114.3 137.16))
-    (stroke (width 0) (type solid) (color 0 0 0 0))
-  )
-  (bus (pts (xy 114.3 137.16) (xy 114.3 142.24))
-    (stroke (width 0) (type solid) (color 0 0 0 0))
-  )
-  (bus (pts (xy 114.3 142.24) (xy 114.3 147.32))
-    (stroke (width 0) (type solid) (color 0 0 0 0))
-  )
-  (bus (pts (xy 114.3 147.32) (xy 114.3 154.94))
-    (stroke (width 0) (type solid) (color 0 0 0 0))
-  )
-  (bus (pts (xy 114.3 154.94) (xy 114.3 160.02))
-    (stroke (width 0) (type solid) (color 0 0 0 0))
-  )
-  (bus (pts (xy 114.3 160.02) (xy 114.3 165.1))
+  (bus (pts (xy 114.3 121.92) (xy 114.3 127))
+    (stroke (width 0) (type solid) (color 0 0 0 0))
+  )
+  (bus (pts (xy 114.3 127) (xy 114.3 129.54))
+    (stroke (width 0) (type solid) (color 0 0 0 0))
+  )
+  (bus (pts (xy 114.3 129.54) (xy 114.3 134.62))
+    (stroke (width 0) (type solid) (color 0 0 0 0))
+  )
+  (bus (pts (xy 114.3 134.62) (xy 114.3 137.16))
+    (stroke (width 0) (type solid) (color 0 0 0 0))
+  )
+  (bus (pts (xy 114.3 137.16) (xy 114.3 139.7))
+    (stroke (width 0) (type solid) (color 0 0 0 0))
+  )
+  (bus (pts (xy 114.3 139.7) (xy 114.3 142.24))
+    (stroke (width 0) (type solid) (color 0 0 0 0))
+  )
+  (bus (pts (xy 114.3 142.24) (xy 114.3 144.78))
+    (stroke (width 0) (type solid) (color 0 0 0 0))
+  )
+  (bus (pts (xy 114.3 144.78) (xy 114.3 147.32))
+    (stroke (width 0) (type solid) (color 0 0 0 0))
+  )
+  (bus (pts (xy 114.3 147.32) (xy 114.3 152.4))
+    (stroke (width 0) (type solid) (color 0 0 0 0))
+  )
+  (bus (pts (xy 114.3 152.4) (xy 114.3 154.94))
+    (stroke (width 0) (type solid) (color 0 0 0 0))
+  )
+  (bus (pts (xy 114.3 154.94) (xy 114.3 157.48))
+    (stroke (width 0) (type solid) (color 0 0 0 0))
+  )
+  (bus (pts (xy 114.3 157.48) (xy 114.3 160.02))
+    (stroke (width 0) (type solid) (color 0 0 0 0))
+  )
+  (bus (pts (xy 114.3 160.02) (xy 114.3 162.56))
+    (stroke (width 0) (type solid) (color 0 0 0 0))
+  )
+  (bus (pts (xy 114.3 162.56) (xy 114.3 165.1))
     (stroke (width 0) (type solid) (color 0 0 0 0))
   )
@@
       (effects (font (size 1.27 1.27)) (justify right))
     )
-    (property "Footprint" "Resistor_SMD:R_0603_1608Metric" (id 2) (at 268.986 151.384 90)
+    (property "Footprint" "Resistor_SMD:R_0402_1005Metric" (id 2) (at 268.986 151.384 90)
       (effects (font (size 1.27 1.27)) hide)
     )
@@
       (effects (font (size 1.27 1.27)) hide)
     )
+    (property "Rated Voltage" "50V" (id 4) (at 74.93 43.18 0)
+      (effects (font (size 1.27 1.27)) hide)
+    )
   )
   (symbol (lib_id "Device:C_Small") (at 86.36 43.18 0) (unit 1)
@@
       (effects (font (size 1.27 1.27)) (justify left))
     )
-    (property "Footprint" "Capacitor_SMD:C_0603_1608Metric" (id 2) (at 268.9352 166.37 0)
-      (effects (font (size 1.27 1.27)) hide)
-    )
+    (property "Footprint" "Capacitor_SMD:C_0402_1005Metric" (id 2) (at 268.9352 166.37 0)
+      (effects (font (size 1.27 1.27)) hide)
+    )

Commit message: Route RGMII signals
Parts:
- removed U401: MIC33050-4YHL, Package_DFN_QFN:HDFN-12-1EP_3x3mm_P0.5mm_EP1.8x1.125mm, symbol MIC33050-4YHL:MIC33050-4YHL
- added L401: 1uH, Inductor_SMD:L_0805_2012Metric, symbol Device:L
- added U401: MIC23050-4YML, Package_DFN_QFN:Micrel_MLF-8-1EP_2x2mm_P0.5mm_EP0.8x1.3mm_ThermalVias, symbol Regulator_Switching:MIC23050-4YML
- C403: value 10u -> 4.7u
Connections:
- net +3V3: now also U401.2 (EN), U401.7 (VIN)
- net CFF: now also U401.5 (CFF)
- net DVDDL: now also L401.2, U401.4 (SNS)
- net GND: now also U401.6 (AGND), U401.8 (PGND)
- new net: L401.1, U401.1 (SW)
- no-connect marks 3 -> 2
Other:
- note added: "Layout note: RGMII signal traces should be length-matched with 50 ohm single-ended impedance."
Changed lines of the file:
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@@
   (junction (at 33.02 36.83) (diameter 1.016) (color 0 0 0 0))
   (junction (at 39.37 36.83) (diameter 1.016) (color 0 0 0 0))
-  (junction (at 53.34 54.61) (diameter 1.016) (color 0 0 0 0))
+  (junction (at 48.26 54.61) (diameter 1.016) (color 0 0 0 0))
+  (junction (at 50.8 54.61) (diameter 1.016) (color 0 0 0 0))
   (junction (at 55.88 54.61) (diameter 1.016) (color 0 0 0 0))
-  (junction (at 58.42 54.61) (diameter 1.016) (color 0 0 0 0))
   (junction (at 74.93 36.83) (diameter 1.016) (color 0 0 0 0))
   (junction (at 74.93 39.37) (diameter 1.016) (color 0 0 0 0))
@@
   (junction (at 327.66 147.32) (diameter 1.016) (color 0 0 0 0))
   (junction (at 330.2 147.32) (diameter 1.016) (color 0 0 0 0))
+  (no_connect (at 208.28 185.42))
   (no_connect (at 208.28 134.62))
-  (no_connect (at 45.72 39.37))
-  (no_connect (at 208.28 185.42))
   (bus_entry (at 114.3 129.54) (size 2.54 2.54)
     (stroke (width 0.1524) (type solid) (color 0 0 0 0))
@@
     (stroke (width 0) (type solid) (color 0 0 0 0))
   )
-  (wire (pts (xy 33.02 54.61) (xy 53.34 54.61))
-    (stroke (width 0) (type solid) (color 0 0 0 0))
-  )
-  (wire (pts (xy 39.37 36.83) (xy 45.72 36.83))
-    (stroke (width 0) (type solid) (color 0 0 0 0))
-  )
-  (wire (pts (xy 39.37 41.91) (xy 39.37 36.83))
-    (stroke (width 0) (type solid) (color 0 0 0 0))
-  )
-  (wire (pts (xy 45.72 41.91) (xy 39.37 41.91))
-    (stroke (width 0) (type solid) (color 0 0 0 0))
-  )
-  (wire (pts (xy 53.34 52.07) (xy 53.34 54.61))
-    (stroke (width 0) (type solid) (color 0 0 0 0))
-  )
-  (wire (pts (xy 53.34 54.61) (xy 55.88 54.61))
-    (stroke (width 0) (type solid) (color 0 0 0 0))
-  )
-  (wire (pts (xy 55.88 52.07) (xy 55.88 54.61))
+  (wire (pts (xy 33.02 54.61) (xy 48.26 54.61))
+    (stroke (width 0) (type solid) (color 0 0 0 0))
+  )
+  (wire (pts (xy 39.37 36.83) (xy 40.64 36.83))
+    (stroke (width 0) (type solid) (color 0 0 0 0))
+  )
+  (wire (pts (xy 39.37 39.37) (xy 39.37 36.83))
+    (stroke (width 0) (type solid) (color 0 0 0 0))
+  )
+  (wire (pts (xy 40.64 39.37) (xy 39.37 39.37))
+    (stroke (width 0) (type solid) (color 0 0 0 0))
+  )
+  (wire (pts (xy 48.26 52.07) (xy 48.26 54.61))
+    (stroke (width 0) (type solid) (color 0 0 0 0))
+  )
+  (wire (pts (xy 48.26 54.61) (xy 50.8 54.61))
+    (stroke (width 0) (type solid) (color 0 0 0 0))
+  )
+  (wire (pts (xy 50.8 52.07) (xy 50.8 54.61))
+    (stroke (width 0) (type solid) (color 0 0 0 0))
+  )
+  (wire (pts (xy 50.8 54.61) (xy 55.88 54.61))
     (stroke (width 0) (type solid) (color 0 0 0 0))
   )
@@
     (stroke (width 0) (type solid) (color 0 0 0 0))
   )
-  (wire (pts (xy 55.88 54.61) (xy 58.42 54.61))
-    (stroke (width 0) (type solid) (color 0 0 0 0))
-  )
-  (wire (pts (xy 58.42 52.07) (xy 58.42 54.61))
-    (stroke (width 0) (type solid) (color 0 0 0 0))
-  )
-  (wire (pts (xy 58.42 54.61) (xy 86.36 54.61))
-    (stroke (width 0) (type solid) (color 0 0 0 0))
-  )
-  (wire (pts (xy 66.04 36.83) (xy 74.93 36.83))
-    (stroke (width 0) (type solid) (color 0 0 0 0))
-  )
-  (wire (pts (xy 66.04 39.37) (xy 74.93 39.37))
-    (stroke (width 0) (type solid) (color 0 0 0 0))
-  )
-  (wire (pts (xy 66.04 41.91) (xy 71.12 41.91))
+  (wire (pts (xy 55.88 54.61) (xy 86.36 54.61))
+    (stroke (width 0) (type solid) (color 0 0 0 0))
+  )
+  (wire (pts (xy 60.96 36.83) (xy 64.77 36.83))
+    (stroke (width 0) (type solid) (color 0 0 0 0))
+  )
+  (wire (pts (xy 60.96 39.37) (xy 74.93 39.37))
+    (stroke (width 0) (type solid) (color 0 0 0 0))
+  )
+  (wire (pts (xy 60.96 41.91) (xy 71.12 41.91))
     (stroke (width 0) (type solid) (color 0 0 0 0))
   )
@@
     (stroke (width 0) (type solid) (color 0 0 0 0))
   )
+  (wire (pts (xy 72.39 36.83) (xy 74.93 36.83))
+    (stroke (width 0) (type solid) (color 0 0 0 0))
+  )
   (wire (pts (xy 74.93 36.83) (xy 74.93 39.37))
     (stroke (width 0) (type solid) (color 0 0 0 0))
@@
   (text "LED_MODE pulled up\nto set single LED mode." (at 96.52 182.88 180)
     (effects (font (size 1.27 1.27)) (justify right bottom))
+  )
+  (text "Layout note:\nRGMII signal traces should be\nlength-matched with 50 ohm\nsingle-ended impedance."
+    (at 99.06 118.11 0)
+    (effects (font (size 1.27 1.27)) (justify left bottom))
   )
   (text "Maybe put ferrites on RGMII lines?" (at 109.22 143.51 180)
@@
     )
     (property "Datasheet" "" (id 3) (at 347.98 76.2 0)
+      (effects (font (size 1.27 1.27)) hide)
+    )
+  )
+  (symbol (lib_id "Device:L") (at 68.58 36.83 90) (unit 1)
+    (in_bom yes) (on_board yes)
+    (property "Reference" "L401" (id 0) (at 68.58 32.1118 90))
+    (property "Value" "1uH" (id 1) (at 68.58 34.417 90))
+    (property "Footprint" "Inductor_SMD:L_0805_2012Metric" (id 2) (at 68.58 36.83 0)
+      (effects (font (size 1.27 1.27)) hide)
+    )
+    (property "Datasheet" "~" (id 3) (at 68.58 36.83 0)
+      (effects (font (size 1.27 1.27)) hide)
+    )
+    (property "Manufacturer" "TDK" (id 4) (at 68.58 36.83 90)
+      (effects (font (size 1.27 1.27)) hide)
+    )
+    (property "Part Number" "MLP2016S1R0MT0S1" (id 5) (at 68.58 36.83 90)
       (effects (font (size 1.27 1.27)) hide)
     )
@@
       (effects (font (size 1.27 1.27)) (justify left))
     )
-    (property "Value" "10u" (id 1) (at 88.6842 44.3293 0)
+    (property "Value" "4.7u" (id 1) (at 88.6968 44.323 0)
       (effects (font (size 1.27 1.27)) (justify left))
     )
@@
     )
   )
-  (symbol (lib_name "MIC33050-4YHL:MIC33050-4YHL_1") (lib_id "MIC33050-4YHL:MIC33050-4YHL") (at 55.88 41.91 0) (unit 1)
-    (in_bom yes) (on_board yes)
-    (property "Reference" "U401" (id 0) (at 55.88 30.0798 0))
-    (property "Value" "MIC33050-4YHL" (id 1) (at 55.88 32.3785 0))
-    (property "Footprint" "Package_DFN_QFN:HDFN-12-1EP_3x3mm_P0.5mm_EP1.8x1.125mm" (id 2) (at 21.59 30.48 0)
-      (effects (font (size 1.27 1.27)) (justify left) hide)
-    )
-    (property "Datasheet" "http://ww1.microchip.com/downloads/en/DeviceDoc/MIC33050-4MHz-Internal-Inductor-PWM-Buck-Power-Module-with-HyperLight-Load-DS20006120A.pdf" (id 3) (at 50.8 38.1 0)
-      (effects (font (size 1.27 1.27)) (justify left) hide)
-    )
-  )
+  (symbol (lib_id "Regulator_Switching:MIC23050-4YML") (at 50.8 41.91 0) (unit 1)
+    (in_bom yes) (on_board yes)
+    (property "Reference" "U401" (id 0) (at 50.8 29.4411 0)
+      (effects (font (size 1.524 1.524)))
+    )
+    (property "Value" "MIC23050-4YML" (id 1) (at 50.8 32.1487 0)
+      (effects (font (size 1.524 1.524)))
+    )
+    (property "Footprint" "Package_DFN_QFN:Micrel_MLF-8-1EP_2x2mm_P0.5mm_EP0.8x1.3mm_ThermalVias" (id 2) (at 55.88 40.64 0)
+      (effects (font (size 1.524 1.524)) (justify left) hide)
+    )
+    (property "Datasheet" "http://ww1.microchip.com/downloads/en/DeviceDoc/mic23050.pdf" (id 3) (at 55.88 45.72 0)
+      (effects (font (size 1.524 1.524)) (justify left) hide)
+    )
+  )

Commit message: Layout Ethernet PHY decoupling capacitors
Parts:
- removed C424: 10u, Capacitor_SMD:C_0603_1608Metric, symbol Device:C_Small
- added C425: 10u, Capacitor_SMD:C_0603_1608Metric, symbol Device:C_Small
- C404: renamed from C405; LCSC Part Number (none) -> C19702; Manufacturer (none) -> Samsung Electro-Mechanics; Part Number (none) -> CL10A106KP8NNNC; Rated Voltage (none) -> 10V; Temperature Coefficient (none) -> X5R
- C405: renamed from C406; footprint Capacitor_SMD:C_0603_1608Metric -> Capacitor_SMD:C_0402_1005Metric; Manufacturer (none) -> Samsung Electro-Mechanics; Part Number (none) -> CL05A106MQ5NUNC; Rated Voltage (none) -> 6.3V; Temperature Coefficient (none) -> X5R
- C406: renamed from C407; footprint Capacitor_SMD:C_0603_1608Metric -> Capacitor_SMD:C_0402_1005Metric; Manufacturer (none) -> Samsung Electro-Mechanics; Part Number (none) -> CL05A106MQ5NUNC; Rated Voltage (none) -> 6.3V; Temperature Coefficient (none) -> X5R
- C407: renamed from C408; Temperature Coefficient (none) -> X7R
- C408: renamed from C409; Temperature Coefficient (none) -> X7R
- C409: renamed from C410; Temperature Coefficient (none) -> X7R
- C410: renamed from C411; Temperature Coefficient (none) -> X7R
- C411: renamed from C412; Temperature Coefficient (none) -> X7R
- C412: renamed from C404; footprint Capacitor_SMD:C_0603_1608Metric -> Capacitor_SMD:C_0402_1005Metric; Manufacturer (none) -> Samsung Electro-Mechanics; Part Number (none) -> CL05A106MQ5NUNC; Rated Voltage (none) -> 6.3V
- C413, C414, C415, C416, C417, C418, C419, C420, C421: Temperature Coefficient (none) -> X7R
- C423: renamed from C429; Temperature Coefficient (none) -> X7R
- C426: renamed from C425; Temperature Coefficient (none) -> X7R
- C427: renamed from C426; Temperature Coefficient (none) -> X7R
- C428: renamed from C427; Temperature Coefficient (none) -> X7R
- C429: renamed from C428; Temperature Coefficient (none) -> X7R
- FB401, FB402, FB403: value 100 ohms -> 120 ohms; footprint Inductor_SMD:L_0402_1005Metric -> Inductor_SMD:L_0603_1608Metric; LCSC Part Number (none) -> C73100; Manufacturer (none) -> Murata Electronics; Part Number (none) -> BLM18PG121SN1D
- renumbered C423 to C424
Connections:
- net AVDDH: now also C425.1
- net GND: now also C425.2
Other:
- moved on the sheet: C412
